Commit message: Fix files for ROS Melodic version

File: quad_description/urdf/kit_c_base.xacro (robot description, xacro)
@@ -36,9 +36,9 @@
       camera_suffix=""
       frame_rate="30"
-      horizontal_fov="2"
+      horizontal_fov="3"
       image_width="1280"
       image_height="720"
       image_format="R8G8B8"
-      min_distance="0.02"
+      min_distance="0.01"
       max_distance="300"
       noise_mean="0.0"
@@ -47,5 +47,6 @@
     >
       <box size="0.2 0.2 0.2" />
-      <origin xyz="0.035 -0.035 0.028" rpy="0 0 0" />
+      <!--origin xyz="0.035 -0.035 0.028" rpy="0 0 0" /-->
+      <origin xyz="0 0 -0.05" rpy="0 1.57 0" />
     </xacro:camera_macro>
   </xacro:if>
